File: project/_uc.kicad_sch (KiCad schematic)
At the start: 35 parts, among them J301 USB_C_Receptacle_USB2.0, SW301 15mm, SW302 15mm, U301 USBLC6-2SC6, U302 esp32-C3FH4X, U303 XL1050, Y301 40MHz

Commit message: fixing CAN level shifting resistors
Parts:
- added R313: 3k, Resistor_SMD:R_0805_2012Metric_Pad1.20x1.40mm_HandSolder, symbol Device:R
- R309: value 4k7 -> 1k5; lcsc# C17673 -> C4310
Connections:
- net GND: now also R313.1
- net RX: now also R313.2
Changed lines of the file:
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@@
   (title_block
     (title "WormControl-Input32-ControlBoard")
-    (date "2026-03-20")
+    (date "2026-08-10")
     (rev "0.2")
     (company "makerspace.lt")
@@
   )
   (junction (at 201.93 133.35) (diameter 0) (color 0 0 0 0)
+  )
+  (junction (at 184.15 133.35) (diameter 0) (color 0 0 0 0)
   )
   (junction (at 148.59 48.26) (diameter 0) (color 0 0 0 0)
@@
     (stroke (width 0) (type default) (color 0 0 0 0))
   )
+  (wire (pts (xy 181.61 133.35) (xy 184.15 133.35))
+    (stroke (width 0) (type default) (color 0 0 0 0))
+  )
   (wire (pts (xy 148.59 48.26) (xy 138.43 48.26))
     (stroke (width 0) (type default) (color 0 0 0 0))
@@
   (hierarchical_label "CLOCK" (shape output) (at 189.23 104.14 0)
     (effects (font (size 1.27 1.27)) (justify left))
+  )
+  (hierarchical_label "GND" (shape bidirectional) (at 173.99 133.35 180)
+    (effects (font (size 1.27 1.27)) (justify right))
   )
   (hierarchical_label "GND" (shape bidirectional) (at 231.14 124.46 0)
@@
     (pin "2")
   )
+  (symbol (lib_id "Device:R") (at 177.8 133.35 90) (unit 1)
+    (in_bom yes) (on_board yes)
+    (property "Reference" "R313" (id 0) (at 177.8 135.89 90))
+    (property "Value" "3k" (id 1) (at 177.8 133.35 90))
+    (property "Footprint" "Resistor_SMD:R_0805_2012Metric_Pad1.20x1.40mm_HandSolder" (id 2) (at 177.8 135.128 90)
+      (effects (font (size 1.27 1.27)) hide)
+    )
+    (property "Datasheet" "~" (id 3) (at 177.8 133.35 0)
+      (effects (font (size 1.27 1.27)) hide)
+    )
+    (property "jlc-part-type" "B" (id 4) (at 177.8 133.35 0)
+      (effects (font (size 1.27 1.27)) hide)
+    )
+    (property "lcsc#" "C17661" (id 5) (at 177.8 133.35 0)
+      (effects (font (size 1.27 1.27)) hide)
+    )
+    (pin "1")
+    (pin "2")
+  )
   (symbol (lib_id "Device:D_Schottky") (at 53.34 135.89 270) (unit 1)
     (in_bom yes) (on_board yes)
@@
     (in_bom yes) (on_board yes)
     (property "Reference" "R309" (id 0) (at 189.23 135.89 90))
-    (property "Value" "4k7" (id 1) (at 189.23 133.35 90))
+    (property "Value" "1k5" (id 1) (at 189.23 133.35 90))
     (property "Footprint" "Resistor_SMD:R_0805_2012Metric_Pad1.20x1.40mm_HandSolder" (id 2) (at 189.23 135.128 90)
       (effects (font (size 1.27 1.27)) hide)
@@
       (effects (font (size 1.27 1.27)) hide)
     )
-    (property "lcsc#" "C17673" (id 5) (at 189.23 133.35 0)
-      (effects (font (size 1.27 1.27)) hide)
-    )
+    (property "lcsc#" "C4310" (id 5) (at 189.23 133.35 0)
+      (effects (font (size 1.27 1.27)) hide)
+    )
